Commit message: me lo paso a local, odio trabajar en este ordenador

File: practica 1/ramp.urdf (robot description, URDF)
Before this commit: robot ramp, 1 links, 0 joints
Links:
- added link ramp0_link, mass 1.0; collision box size=2 3.35 0.1; visual box size=2 3.35 0.1
Joints:
- added joint base_to_ramp0: type fixed, parent base_link, child ramp0_link, origin xyz=0 2 0.75, limit lower=-0.14 upper=0.14 effort=10.0 velocity=0.5

Commit message: Entendido edición de origenes de joints

File: practica 1/ramp.urdf (robot description, URDF)
Before this commit: robot ramp, 2 links, 1 joints
Links:
- added link rampf_link, mass 1.0; collision box size=2 3.35 0.07; visual box size=2 3.35 0.07
- link ramp0_link: geometry collision box size=2 3.35 0.07; visual box size=2 3.35 0.07
Joints:
- added joint base_to_rampf: type fixed, parent base_link, child rampf_link, origin xyz=0 3.45 0 rpy=-0.4636 0 0, limit lower=-0.14 upper=0.14 effort=10.0 velocity=0.5
- joint base_to_ramp0: origin xyz=0 2 0.75 -> xyz=0 -3.45 0 rpy=0.4636 0 0
