Commit message: Finished structures

File: practica 1/bar.urdf (robot description, URDF)
Before this commit: robot finish_line, 2 links, 1 joints
Links:
- link base_link: geometry collision box size=0.1 0.1 0.6; visual box size=0.1 0.1 0.6
Joints:
- joint base_to_body: origin xyz=0 0 0.14493 -> xyz=0 0 0.02

File: practica 1/finish_line.urdf (robot description, URDF)
Before this commit: robot finish_line, 1 links, 0 joints
Links:
- link base_link: geometry collision box size=3 1 0.01; visual box size=3 1 0.01

File: practica 1/ramp.urdf (robot description, URDF)
Before this commit: robot ramp, 3 links, 2 joints
Links:
- link base_link: geometry collision box size=2 4 1.5; visual box size=2 4 1.5
- link ramp0_link: geometry collision box size=2 3.35 0.001; visual box size=2 3.35 0.001
- link rampf_link: geometry collision box size=2 3.35 0.001; visual box size=2 3.35 0.001
