Commit message: tiny changes

File: practica 1/FASE_1/bar.urdf (robot description, URDF)
Before this commit: robot bar, 2 links, 1 joints
Links:
- link base_link: mass 1.0 -> None
Joints:
- joint base_to_body: limit lower=0 upper=1.5708 effort=10.0 velocity=0.5 -> lower=1.5708 upper=0 effort=10.0 velocity=0.5
