Commit message: Last changes

File: practica 1/FASE_3/3.2_dynamics/ramp.urdf (robot description, URDF)
Before this commit: robot arm_robot, 3 links, 2 joints
Links:
- removed link arm_link
- removed link body_link
- added link ramp0_link, mass 1.0; collision box size=2 3.35 0.001; visual box size=2 3.35 0.001
- added link rampf_link, mass 1.0; collision box size=2 3.35 0.001; visual box size=2 3.35 0.001
- link base_link: geometry collision box size=2 4 1.5; visual box size=2 4 1.5
Joints:
- removed joint base_to_body
- removed joint body_to_arm
- added joint base_to_ramp0: type fixed, parent base_link, child ramp0_link, origin xyz=0 -3.45 0 rpy=0.4636 0 0, limit lower=-0.14 upper=0.14 effort=10.0 velocity=0.5
- added joint base_to_rampf: type fixed, parent base_link, child rampf_link, origin xyz=0 3.45 0 rpy=-0.4636 0 0, limit lower=-0.14 upper=0.14 effort=10.0 velocity=0.5

File: practica 1/FASE_3/3.3_inertial/bar.urdf (robot description, URDF)
Before this commit: robot bar, 2 links, 1 joints
Links:
- added link world
- link base_link: mass 1.0 -> None
- link body_link: mass None -> 5.0
Joints:
- added joint fixed: type fixed, parent world, child base_link, origin xyz=0 0 0.3
- joint base_to_body: limit lower=-0.14 upper=0.14 effort=10.0 velocity=0.5 -> lower=0 upper=3.14 effort=10.0 velocity=0.5

File: practica 1/FASE_4/bar.urdf (robot description, URDF)
Before this commit: robot bar, 3 links, 2 joints
Links:
- link body_link: mass None -> 5.0
Joints:
- joint base_to_body: limit lower=0 upper=1.5708 effort=10.0 velocity=0.5 -> lower=0 upper=3.14 effort=10.0 velocity=0.5
