Commit message: chassis in pybullet

File: BLENDER/class_chassis/test/urdf/test.urdf (robot description, URDF)
Before this commit: robot test, 3 links, 2 joints
Links:
- link axis_link: mass None -> 6.00000; geometry collision box size=0.19835 2.51094 0.19658; visual box size=0.20222 0.20000 2.50000
- link left_wheel_link: mass None -> 1.00000; geometry collision mesh filename=../meshes/dae/Torus.dae scale=0.29646 0.29646 0.29646; visual mesh filename=../meshes/dae/Torus.dae scale=0.29646 0.29646 0.29646
- link right_wheel_link: mass None -> 1.00000; geometry collision mesh filename=../meshes/dae/Torus.001.dae scale=0.29646 0.29646 0.29646; visual mesh filename=../meshes/dae/Torus.001.dae scale=0.29646 0.29646 0.29646
