Commit message: Sbs? la cosa es que yo cuando leí cubo entendñi pues un cubo de toda la vida como el de minecraft. bueno pues mi cara cuando los profesores me dicen que se refieren a CUBOS prismas tetraedros fue interesante. red in the face.

File: practica2/pybullet/cubo/urdf/cubo.urdf (robot description, URDF)
Before this commit: robot cubo, 1 links, 0 joints
Links:
- link base_link: mass 1.0 -> 2.0; geometry collision box size=0.5 0.5 0.5; visual box size=0.5 0.5 0.5
