Commit message: fixed pinza

File: practica2/pybullet/rover/urdf/rover.urdf (robot description, URDF)
Before this commit: robot rover, 17 links, 16 joints
Links:
- added link pris_link4.001_link, mass 0.50000; collision box size=0.02510 0.06000 0.09410; visual mesh filename=../meshes/dae/Cylinder.009.dae scale=0.03922 0.03922 0.61477
- added link pris_link4.002_link, mass 0.50000; collision box size=0.02510 0.06000 0.09410; visual mesh filename=../meshes/dae/Cylinder.010.dae scale=0.03922 0.03922 0.61477
- link pris_link4_link: mass 1.00000 -> 4.00000
Joints:
- added joint pris_link4.001_link_joint: type prismatic, parent pris_link4_link, child pris_link4.001_link, origin xyz=0.34912 0.00059 0.07033 rpy=3.14159 -1.57080 -3.14159, axis 0.00000 0.00000 1.00000, limit lower=0.00000 upper=0.20000 effort=0.00000 velocity=0.00000
- added joint pris_link4.002_link_joint: type prismatic, parent pris_link4_link, child pris_link4.002_link, origin xyz=-0.34568 0.00059 0.07033 rpy=0.00000 1.57080 0.00000, axis 0.00000 0.00000 1.00000, limit lower=0.00000 upper=0.20000 effort=0.00000 velocity=0.00000
- joint pris_link4_link_joint: limit lower=-1.00000 upper=3.14000 effort=0.00000 velocity=0.00000 -> lower=-0.50000 upper=3.00000 effort=0.00000 velocity=0.00000; origin xyz=0.00000 -0.00000 0.00000 rpy=-3.14159 -0.00000 -1.57080 -> xyz=-0.00000 -0.00000 -0.00000 rpy=3.14159 -0.00000 1.57080

Commit message: make it 58

File: practica2/pybullet/rover/urdf/rover.urdf (robot description, URDF)
Before this commit: robot rover, 19 links, 18 joints
Links:
- added link Cube.001_link, mass 0.00100; collision box size=0.04158 0.98771 0.10979; visual box size=0.04657 0.98760 0.09602
- added link Cube.002_link, mass 0.00100; collision box size=0.05301 0.92029 0.10866; visual box size=0.04657 0.89445 0.09602
- added link Cube_link, mass 0.00100; collision box size=0.06923 0.98010 0.10221; visual box size=0.04657 0.98760 0.09602
- link chassis_link: mass 20.00000 -> 0.00100
- link pris_link4_link: mass 4.00000 -> 0.00100
Joints:
- added joint Cube.001_link_joint: type fixed, parent chassis_link, child Cube.001_link, origin xyz=-0.62849 1.02834 0.42156 rpy=0.00000 0.00000 3.14159
- added joint Cube.002_link_joint: type fixed, parent chassis_link, child Cube.002_link, origin xyz=-0.01153 0.38661 0.42391 rpy=0.00000 0.00000 1.57080, axis 0.00000 0.00000 1.00000
- added joint Cube_link_joint: type fixed, parent chassis_link, child Cube_link, origin xyz=0.62053 1.02834 0.42156 rpy=0.00000 0.00000 3.14159
- joint pris_link4.001_link_joint: origin xyz=0.34912 0.00059 0.07033 rpy=3.14159 -1.57080 -3.14159 -> xyz=0.34912 0.00059 0.07033 rpy=-3.14159 -1.57080 3.14159
- joint pris_link4.002_link_joint: origin xyz=-0.34568 0.00059 0.07033 rpy=0.00000 1.57080 0.00000 -> xyz=-0.34568 0.00059 0.07033 rpy=-0.00000 1.57080 0.00000
- joint pris_link4_link_joint: limit lower=-0.50000 upper=3.00000 effort=0.00000 velocity=0.00000 -> lower=-0.20000 upper=2.30000 effort=0.00000 velocity=0.00000
- joint rot_link4_link_joint: origin xyz=-0.99849 0.00559 -0.52727 rpy=0.00000 -0.00000 0.00000 -> xyz=-0.99849 0.00559 -0.52727 rpy=0.00000 0.00000 -0.00000

Commit message: more space for cube. changes to code, still too difficult to work on. no puedo mas

File: practica2/pybullet/rover/urdf/rover.urdf (robot description, URDF)
Before this commit: robot rover, 22 links, 21 joints
Links:
- link chassis_link: geometry collision box size=1.07593 0.96827 0.25516; collision box size=1.46371 0.45353 0.10904
Joints:
- joint Cube.001_link_joint: origin xyz=-0.62849 1.02834 0.42156 rpy=0.00000 0.00000 3.14159 -> xyz=-0.78494 1.00818 0.42156 rpy=0.00000 0.00000 3.14159
- joint Cube_link_joint: origin xyz=0.62053 1.02834 0.42156 rpy=0.00000 0.00000 3.14159 -> xyz=0.76908 0.97227 0.42156 rpy=0.00000 0.00000 3.14159
