Commit message: scara and gripper

File: practica3/rover_kachau/urdf/arm/gripper.urdf.xacro (robot description, xacro)
@@ -1,11 +1,4 @@
 <?xml version="1.0"?>
 <robot xmlns:xacro="http://www.ros.org/wiki/xacro">
-  <joint name="rot_link4_link_joint" type="continuous">
-    <limit effort="0.00000" velocity="0.00000"/>
-    <origin rpy="0.00000 0.00000 -0.00000" xyz="-0.99849 0.00559 -0.52727"/>
-    <parent link="link3_link"/>
-    <child link="rot_link4_link"/>
-    <axis xyz="0.00000 0.00000 1.00000"/>
-  </joint>
   <joint name="pris_link4_link_joint" type="prismatic">
     <limit lower="-0.20000" upper="2.30000" effort="0.00000" velocity="0.00000"/>
@@ -29,24 +22,4 @@
     <axis xyz="0.00000 0.00000 1.00000"/>
   </joint>
-  <link name="rot_link4_link">
-    <collision name="rot_link4_collision">
-      <origin rpy="0.00000 0.00000 -0.00000" xyz="0.00000 -0.00000 0.31437"/>
-      <geometry>
-        <cylinder radius="0.07101" length="0.27439"/>
-      </geometry>
-    </collision>
-    <inertial>
-      <inertia ixx="0.00404" ixy="0.00000" ixz="0.00000" iyy="0.00404" iyz="0.00000" izz="0.00126"/>
-      <origin rpy="0.00000 0.00000 0.00000" xyz="0.00000 -0.00000 0.31363"/>
-      <mass value="0.50000"/>
-    </inertial>
-    <visual name="rot_link4">
-      <material name="Material.017"/>
-      <origin rpy="-0.00000 -0.00000 0.00000" xyz="-0.00000 -0.00000 0.31363"/>
-      <geometry>
-        <cylinder radius="0.07102" length="0.28609"/>
-      </geometry>
-    </visual>
-  </link>
   <link name="pris_link4_link">
     <collision name="pris_link4_collision">
@@ -115,6 +88,3 @@
     <color rgba="0.00000 0.00392 1.00000 1.00000"/>
   </material>
-  <material name="Material.017">
-    <color rgba="0.00000 0.00000 0.00000 1.00000"/>
-  </material>
 </robot>

Commit message: gripper upside down. scara_base down. must fix

File: practica3/rover_kachau/urdf/arm/gripper.urdf.xacro (robot description, xacro)
@@ -4,5 +4,5 @@
     <joint name="${prefix}_gripper_mount_joint" type="fixed">
       <parent link="${parent_link}"/>
-      <child link="${prefix}_rot_link4_link"/>
+      <child link="${prefix}_pris_link4_link"/>
       <origin xyz="0 0 0" rpy="0 0 0"/>
     </joint>
@@ -32,5 +32,5 @@
         <origin rpy="3.14159 0.00000 -3.14159" xyz="-0.00000 0.00000 -0.00000"/>
         <geometry>
-          <mesh filename="$(find rover_kachau)/meshes/dae/Cylinder.013.dae" scale="0.03922 0.03922 0.61477"/>
+          <mesh filename="package://rover_kachau/meshes/dae/Cylinder.013.dae" scale="0.03922 0.03922 0.61477"/>
         </geometry>
       </collision>
@@ -44,5 +44,5 @@
         <origin rpy="3.14159 0.00000 3.14159" xyz="-0.00000 0.00000 -0.00000"/>
         <geometry>
-          <mesh filename="$(find rover_kachau)/meshes/dae/Cylinder.013.dae" scale="0.03922 0.03922 0.61477"/>
+          <mesh filename="package://rover_kachau/meshes/dae/Cylinder.013.dae" scale="0.03922 0.03922 0.61477"/>
         </geometry>
       </visual>
@@ -64,5 +64,5 @@
         <origin rpy="-0.00000 -1.57080 0.00000" xyz="-0.00000 -0.00000 -0.00000"/>
         <geometry>
-          <mesh filename="$(find rover_kachau)/meshes/dae/Cylinder.009.dae" scale="0.03922 0.03922 0.61477"/>
+          <mesh filename="package://rover_kachau/meshes/dae/Cylinder.009.dae" scale="0.03922 0.03922 0.61477"/>
         </geometry>
       </visual>
@@ -84,5 +84,5 @@
         <origin rpy="0.00000 1.57080 0.00000" xyz="0.00000 0.00000 -0.00000"/>
         <geometry>
-          <mesh filename="$(find rover_kachau)/meshes/dae/Cylinder.010.dae" scale="0.03922 0.03922 0.61477"/>
+          <mesh filename="package://rover_kachau/meshes/dae/Cylinder.010.dae" scale="0.03922 0.03922 0.61477"/>
         </geometry>
       </visual>

File: practica3/rover_kachau/urdf/arm/scara.urdf.xacro (robot description, xacro)
@@ -145,5 +145,5 @@
         <origin rpy="3.14159 0.00000 -3.14159" xyz="-0.00000 0.00000 -0.00000"/>
         <geometry>
-          <mesh filename="$(find rover_kachau)/meshes/dae/Cylinder.013.dae" scale="0.03922 0.03922 0.61477"/>
+          <mesh filename="package://rover_kachau/meshes/dae/Cylinder.013.dae" scale="0.03922 0.03922 0.61477"/>
         </geometry>
       </collision>
@@ -157,5 +157,5 @@
         <origin rpy="3.14159 0.00000 3.14159" xyz="-0.00000 0.00000 -0.00000"/>
         <geometry>
-          <mesh filename="$(find rover_kachau)/meshes/dae/Cylinder.013.dae" scale="0.03922 0.03922 0.61477"/>
+          <mesh filename="package://rover_kachau/meshes/dae/Cylinder.013.dae" scale="0.03922 0.03922 0.61477"/>
         </geometry>
       </visual>

File: practica3/rover_kachau/urdf/tank/rover_tank.urdf.xacro (robot description, xacro)
@@ -2,21 +2,21 @@
 <robot name="rover" xmlns:xacro="http://www.ros.org/wiki/xacro">
   <xacro:macro name="tank" params="prefix parent_link">
-    <joint name="{prefix}_Cube.001_link_joint" type="fixed">
+    <joint name="${prefix}_Cube.001_link_joint" type="fixed">
       <origin rpy="0.00000 0.00000 3.14159" xyz="-0.78494 1.00818 0.42156"/>
-      <parent link="{parent_link}"/>
-      <child link="{prefix}_Cube.001_link"/>
+      <parent link="${parent_link}"/>
+      <child link="${prefix}_Cube.001_link"/>
     </joint>
-    <joint name="{prefix}_Cube.002_link_joint" type="fixed">
+    <joint name="${prefix}_Cube.002_link_joint" type="fixed">
       <origin rpy="0.00000 0.00000 1.57080" xyz="-0.01153 0.38661 0.42391"/>
-      <parent link="{parent_link}"/>
-      <child link="{prefix}_Cube.002_link"/>
+      <parent link="${parent_link}"/>
+      <child link="${prefix}_Cube.002_link"/>
       <axis xyz="0.00000 0.00000 1.00000"/>
     </joint>
-    <joint name="{prefix}_Cube_link_joint" type="fixed">
+    <joint name="${prefix}_Cube_link_joint" type="fixed">
       <origin rpy="0.00000 0.00000 3.14159" xyz="0.76908 0.97227 0.42156"/>
-      <parent link="{parent_link}"/>
-      <child link="{prefix}_Cube_link"/>
+      <parent link="${parent_link}"/>
+      <child link="${prefix}_Cube_link"/>
     </joint>
-    <link name="{prefix}_Cube.001_link">
+    <link name="${prefix}_Cube.001_link">
       <collision name="Cube.001_collision">
         <origin rpy="0.00000 0.00000 0.00000" xyz="0.00000 0.00000 0.00000"/>
@@ -38,5 +38,5 @@
       </visual>
     </link>
-    <link name="{prefix}_Cube.002_link">
+    <link name="${prefix}_Cube.002_link">
       <collision name="Cube.002_collision">
         <origin rpy="0.00000 0.00000 0.00000" xyz="0.00000 0.00000 0.00000"/>
@@ -58,5 +58,5 @@
       </visual>
     </link>
-    <link name="{prefix}_Cube_link">
+    <link name="${prefix}_Cube_link">
       <collision name="Cube_collision">
         <origin rpy="0.00000 0.00000 0.00000" xyz="0.00000 0.00000 0.00000"/>

Commit message: base del scara arreglado. gripper sigue upside down. ademas el codigo no está bien pensando para una macro, pero es que no me da tiempo

File: practica3/rover_kachau/urdf/arm/gripper.urdf.xacro (robot description, xacro)
@@ -5,5 +5,5 @@
       <parent link="${parent_link}"/>
       <child link="${prefix}_pris_link4_link"/>
-      <origin xyz="0 0 0" rpy="0 0 0"/>
+      <origin xyz="0 0 0" rpy="3.14159 0 0"/>
     </joint>
     <joint name="${prefix}_pris_link4_link_joint" type="prismatic">

File: practica3/rover_kachau/urdf/arm/scara.urdf.xacro (robot description, xacro)
@@ -5,5 +5,5 @@
       <parent link="${parent_link}"/>
       <child link="${prefix}_scara_base_link"/>
-      <origin xyz="0 0 0" rpy="0 0 0"/>
+      <origin xyz="${arm_offset_x} 0 0.55" rpy="0 0 0"/>
     </joint>
     <joint name="${prefix}_link1_link_joint" type="fixed">
