Commit message: followed class tutorial for transmission and gazebo reference

File: practica3/rover_kachau/urdf/wheels/rover_wheel.urdf.xacro (robot description, xacro)
@@ -130,4 +130,15 @@
           <mesh filename="package://rover_kachau/meshes/dae/Cylinder.002.dae" scale="1.00000 1.00000 1.00000"/>
         </geometry>
+        <surface>
+          <friction>
+            <ode>
+              <mu>1.000000</mu>
+              <mu2>1.000000</mu2>
+              <fdir1>0.000000 0.000000 1.000000</fdir1>
+              <slip1>0.50000<slip1>
+              <slip2>0.50000<slip2>
+            </ode>
+          </friction>
+        </surface>
       </collision>
       <inertial>
@@ -170,4 +181,15 @@
           <mesh filename="package://rover_kachau/meshes/dae/Cylinder.004.dae" scale="1.00000 1.00000 1.00000"/>
         </geometry>
+        <surface>
+          <friction>
+            <ode>
+              <mu>1.000000</mu>
+              <mu2>1.000000</mu2>
+              <fdir1>0.000000 0.000000 1.000000</fdir1>
+              <slip1>0.50000<slip1>
+              <slip2>0.50000<slip2>
+            </ode>
+          </friction>
+        </surface>
       </collision>
       <inertial>
@@ -210,4 +232,15 @@
           <mesh filename="package://rover_kachau/meshes/dae/Cylinder.001.dae" scale="1.00000 1.00000 1.00000"/>
         </geometry>
+        <surface>
+          <friction>
+            <ode>
+              <mu>1.000000</mu>
+              <mu2>1.000000</mu2>
+              <fdir1>0.000000 0.000000 1.000000</fdir1>
+              <slip1>0.50000<slip1>
+              <slip2>0.50000<slip2>
+            </ode>
+          </friction>
+        </surface>
       </collision>
       <inertial>
@@ -250,4 +283,15 @@
           <mesh filename="package://rover_kachau/meshes/dae/Cylinder.003.dae" scale="1.00000 1.00000 1.00000"/>
         </geometry>
+        <surface>
+          <friction>
+            <ode>
+              <mu>1.000000</mu>
+              <mu2>1.000000</mu2>
+              <fdir1>0.000000 0.000000 1.000000</fdir1>
+              <slip1>0.50000<slip1>
+              <slip2>0.50000<slip2>
+            </ode>
+          </friction>
+        </surface>
       </collision>
       <inertial>
@@ -264,4 +308,61 @@
       </visual>
     </link>
+    <!-- Añadimos transmission para juntar todas as joints -->
+    <transmission name="${prefix}_frontL_trans">
+      <type>transmission_interface/SimpleTransmission</type>
+      <joint name="${prefix}_frontL_link_joint">
+        <hardwareInterface>hardware_interface/VelocityJointInterface</hardwareInterface>
+      </joint>
+      <actuator name="${prefix}_frontL_motor">
+        <mechanicalReduction>1</mechanicalReduction>
+      </actuator>
+    </transmission>
+    <transmission name="${prefix}_frontR_trans">
+      <type>transmission_interface/SimpleTransmission</type>
+      <joint name="${prefix}_frontR_link_joint">
+        <hardwareInterface>hardware_interface/VelocityJointInterface</hardwareInterface>
+      </joint>
+      <actuator name="${prefix}_frontR_motor">
+        <mechanicalReduction>1</mechanicalReduction>
+      </actuator>
+    </transmission>
+    <transmission name="${prefix}_backL_trans">
+      <type>transmission_interface/SimpleTransmission</type>
+      <joint name="${prefix}_backL_link_joint">
+        <hardwareInterface>hardware_interface/VelocityJointInterface</hardwareInterface>
+      </joint>
+      <actuator name="${prefix}_backL_motor">
+        <mechanicalReduction>1</mechanicalReduction>
+      </actuator>
+    </transmission>
+    <transmission name="${prefix}_backR_trans">
+      <type>transmission_interface/SimpleTransmission</type>
+      <joint name="${prefix}_backR_link_joint">
+        <hardwareInterface>hardware_interface/VelocityJointInterface</hardwareInterface>
+      </joint>
+      <actuator name="${prefix}_backR_motor">
+        <mechanicalReduction>1</mechanicalReduction>
+      </actuator>
+    </transmission>
+    <gazebo reference="${prefix}_frontL_link">
+      <mu1>5</mu1>
+      <mu2>5</mu2>
+      <!--kp>2.75e6>/kp>
+      <kd>8.25e1</kd>
+      <fdir1>0 0 0</fdir1>
+      <maxContacts>4</maxContacts-->
+    </gazebo>
+    <gazebo reference="${prefix}_frontR_link">  <!-- corregido -->
+      <mu1>5</mu1>
+      <mu2>5</mu2>
+    </gazebo>
+    <gazebo reference="${prefix}_backL_link">  <!-- corregido -->
+      <mu1>5</mu1>
+      <mu2>5</mu2>
+    </gazebo>
+    <gazebo reference="${prefix}_backR_link">  <!-- corregido -->
+      <mu1>5</mu1>
+      <mu2>5</mu2>
+    </gazebo>
   </xacro:macro>
 </robot>
