Commit message: rviz abre y sliders arreglados. igual deberia cambiar la macro de las ruedas porque son separadas pero es muy comodo que lo abra todo. por ahora no tengo tiempo. add tf, add robot_model descript /robot_description. ademas usar --symlink-install

File: practica3/rover_kachau/robots/robot.urdf.xacro (robot description, xacro)
@@ -23,8 +23,5 @@
 <xacro:robot_base prefix="$(arg prefix)"/>
 <!-- Wheels -->
-<xacro:rover_wheel prefix="front_right_" parent_link="base_link"/>
-<xacro:rover_wheel prefix="back_right_" parent_link="base_link"/>
-<xacro:rover_wheel prefix="front_left_" parent_link="base_link"/>
-<xacro:rover_wheel prefix="back_left_" parent_link="base_link"/>
+<xacro:rover_wheel prefix="rover" parent_link="base_link"/>
 <!-- Arm -->
 <xacro:scara prefix="scara" parent_link="base_link"/>

File: practica3/rover_kachau/urdf/arm/gripper.urdf.xacro (robot description, xacro)
@@ -32,5 +32,5 @@
         <origin rpy="3.14159 0.00000 -3.14159" xyz="-0.00000 0.00000 -0.00000"/>
         <geometry>
-          <mesh filename="../meshes/dae/Cylinder.013.dae" scale="0.03922 0.03922 0.61477"/>
+          <mesh filename="$(find rover_kachau)/meshes/dae/Cylinder.013.dae" scale="0.03922 0.03922 0.61477"/>
         </geometry>
       </collision>
@@ -44,5 +44,5 @@
         <origin rpy="3.14159 0.00000 3.14159" xyz="-0.00000 0.00000 -0.00000"/>
         <geometry>
-          <mesh filename="../meshes/dae/Cylinder.013.dae" scale="0.03922 0.03922 0.61477"/>
+          <mesh filename="$(find rover_kachau)/meshes/dae/Cylinder.013.dae" scale="0.03922 0.03922 0.61477"/>
         </geometry>
       </visual>
@@ -64,5 +64,5 @@
         <origin rpy="-0.00000 -1.57080 0.00000" xyz="-0.00000 -0.00000 -0.00000"/>
         <geometry>
-          <mesh filename="../meshes/dae/Cylinder.009.dae" scale="0.03922 0.03922 0.61477"/>
+          <mesh filename="$(find rover_kachau)/meshes/dae/Cylinder.009.dae" scale="0.03922 0.03922 0.61477"/>
         </geometry>
       </visual>
@@ -84,5 +84,5 @@
         <origin rpy="0.00000 1.57080 0.00000" xyz="0.00000 0.00000 -0.00000"/>
         <geometry>
-          <mesh filename="../meshes/dae/Cylinder.010.dae" scale="0.03922 0.03922 0.61477"/>
+          <mesh filename="$(find rover_kachau)/meshes/dae/Cylinder.010.dae" scale="0.03922 0.03922 0.61477"/>
         </geometry>
       </visual>

File: practica3/rover_kachau/urdf/arm/scara.urdf.xacro (robot description, xacro)
@@ -145,5 +145,5 @@
         <origin rpy="3.14159 0.00000 -3.14159" xyz="-0.00000 0.00000 -0.00000"/>
         <geometry>
-          <mesh filename="../meshes/dae/Cylinder.013.dae" scale="0.03922 0.03922 0.61477"/>
+          <mesh filename="$(find rover_kachau)/meshes/dae/Cylinder.013.dae" scale="0.03922 0.03922 0.61477"/>
         </geometry>
       </collision>
@@ -157,5 +157,5 @@
         <origin rpy="3.14159 0.00000 3.14159" xyz="-0.00000 0.00000 -0.00000"/>
         <geometry>
-          <mesh filename="../meshes/dae/Cylinder.013.dae" scale="0.03922 0.03922 0.61477"/>
+          <mesh filename="$(find rover_kachau)/meshes/dae/Cylinder.013.dae" scale="0.03922 0.03922 0.61477"/>
         </geometry>
       </visual>

File: practica3/rover_kachau/urdf/base/robot_base.urdf.xacro (robot description, xacro)
@@ -48,5 +48,5 @@
         <origin rpy="0.00000 0.00000 0.00000" xyz="0.00000 0.00000 0.00000"/>
         <geometry>
-          <mesh filename="../meshes/dae/Cube.001.dae" scale="1.00000 1.00000 1.00000"/>
+          <mesh filename="$(find rover_kachau)/meshes/dae/Cube.001.dae" scale="1.00000 1.00000 1.00000"/>
         </geometry>
       </visual>

File: practica3/rover_kachau/urdf/wheels/rover_wheel.urdf.xacro (robot description, xacro)
@@ -128,5 +128,5 @@
         <origin rpy="0.01967 0.01541 -0.18756" xyz="0.00000 -0.00000 -0.00000"/>
         <geometry>
-          <mesh filename="../meshes/dae/Cylinder.002.dae" scale="1.00000 1.00000 1.00000"/>
+          <mesh filename="$(find rover_kachau)/meshes/dae/Cylinder.002.dae" scale="1.00000 1.00000 1.00000"/>
         </geometry>
       </collision>
@@ -140,5 +140,5 @@
         <origin rpy="-0.00000 0.00000 0.00000" xyz="-0.00000 -0.00000 -0.00000"/>
         <geometry>
-          <mesh filename="../meshes/dae/Cylinder.007.dae" scale="1.00000 1.00000 1.00000"/>
+          <mesh filename="$(find rover_kachau)/meshes/dae/Cylinder.007.dae" scale="1.00000 1.00000 1.00000"/>
         </geometry>
       </visual>
@@ -168,5 +168,5 @@
         <origin rpy="0.01967 0.01541 -0.18756" xyz="0.00000 -0.00000 -0.00000"/>
         <geometry>
-          <mesh filename="../meshes/dae/Cylinder.004.dae" scale="1.00000 1.00000 1.00000"/>
+          <mesh filename="$(find rover_kachau)/meshes/dae/Cylinder.004.dae" scale="1.00000 1.00000 1.00000"/>
         </geometry>
       </collision>
@@ -180,5 +180,5 @@
         <origin rpy="-0.00000 -0.00000 0.00000" xyz="0.00000 -0.00000 0.00000"/>
         <geometry>
-          <mesh filename="../meshes/dae/Cylinder.008.dae" scale="1.00000 1.00000 1.00000"/>
+          <mesh filename="$(find rover_kachau)/meshes/dae/Cylinder.008.dae" scale="1.00000 1.00000 1.00000"/>
         </geometry>
       </visual>
@@ -208,5 +208,5 @@
         <origin rpy="0.01967 0.01541 -0.18756" xyz="-0.00000 0.00000 -0.00000"/>
         <geometry>
-          <mesh filename="../meshes/dae/Cylinder.001.dae" scale="1.00000 1.00000 1.00000"/>
+          <mesh filename="$(find rover_kachau)/meshes/dae/Cylinder.001.dae" scale="1.00000 1.00000 1.00000"/>
         </geometry>
       </collision>
@@ -220,5 +220,5 @@
         <origin rpy="-0.00000 0.00000 0.00000" xyz="-0.00000 0.00000 -0.00000"/>
         <geometry>
-          <mesh filename="../meshes/dae/Cylinder.005.dae" scale="1.00000 1.00000 1.00000"/>
+          <mesh filename="$(find rover_kachau)/meshes/dae/Cylinder.005.dae" scale="1.00000 1.00000 1.00000"/>
         </geometry>
       </visual>
@@ -248,5 +248,5 @@
         <origin rpy="0.01967 0.01541 -0.18756" xyz="0.00000 0.00000 -0.00000"/>
         <geometry>
-          <mesh filename="../meshes/dae/Cylinder.003.dae" scale="1.00000 1.00000 1.00000"/>
+          <mesh filename="$(find rover_kachau)/meshes/dae/Cylinder.003.dae" scale="1.00000 1.00000 1.00000"/>
         </geometry>
       </collision>
@@ -260,5 +260,5 @@
         <origin rpy="-0.00000 0.00000 0.00000" xyz="0.00000 0.00000 0.00000"/>
         <geometry>
-          <mesh filename="../meshes/dae/Cylinder.006.dae" scale="1.00000 1.00000 1.00000"/>
+          <mesh filename="$(find rover_kachau)/meshes/dae/Cylinder.006.dae" scale="1.00000 1.00000 1.00000"/>
         </geometry>
       </visual>

Commit message: find for wheels and chassis doesnt work, ask teachers. about to fix the tank not showing

File: practica3/rover_kachau/robots/robot.urdf.xacro (robot description, xacro)
@@ -23,7 +23,9 @@
 <xacro:robot_base prefix="$(arg prefix)"/>
 <!-- Wheels -->
-<xacro:rover_wheel prefix="rover" parent_link="base_link"/>
+<xacro:rover_wheel prefix="wheels_" parent_link="base_link"/>
+<!-- Tank -->
+<xacro:tank prefix="tank_" parent_link="base_link"/>
 <!-- Arm -->
-<xacro:scara prefix="scara" parent_link="base_link"/>
+<xacro:scara prefix="" parent_link="base_link"/>
 <!--
 <xacro:include filename="$(find rover_kachau)/urdf/ros2_control.urdf.xacro"/>

File: practica3/rover_kachau/urdf/base/robot_base.urdf.xacro (robot description, xacro)
@@ -45,9 +45,11 @@
       </inertial>
       <visual name="chassis">
-        <material name="Material.001"/>
-        <origin rpy="0.00000 0.00000 0.00000" xyz="0.00000 0.00000 0.00000"/>
+        <origin rpy="0 0 0" xyz="0 0 0"/>
         <geometry>
-          <mesh filename="$(find rover_kachau)/meshes/dae/Cube.001.dae" scale="1.00000 1.00000 1.00000"/>
+          <mesh filename="package://rover_kachau/meshes/dae/Cube.001.dae" scale="1.0 1.0 1.0"/>
         </geometry>
+        <material name="chassis_mat">
+          <color rgba="0.5 0.5 0.5 1"/>
+        </material>
       </visual>
     </link>

File: practica3/rover_kachau/urdf/wheels/rover_wheel.urdf.xacro (robot description, xacro)
@@ -128,5 +128,5 @@
         <origin rpy="0.01967 0.01541 -0.18756" xyz="0.00000 -0.00000 -0.00000"/>
         <geometry>
-          <mesh filename="$(find rover_kachau)/meshes/dae/Cylinder.002.dae" scale="1.00000 1.00000 1.00000"/>
+          <mesh filename="package://rover_kachau/meshes/dae/Cylinder.002.dae" scale="1.00000 1.00000 1.00000"/>
         </geometry>
       </collision>
@@ -140,5 +140,5 @@
         <origin rpy="-0.00000 0.00000 0.00000" xyz="-0.00000 -0.00000 -0.00000"/>
         <geometry>
-          <mesh filename="$(find rover_kachau)/meshes/dae/Cylinder.007.dae" scale="1.00000 1.00000 1.00000"/>
+          <mesh filename="package://rover_kachau/meshes/dae/Cylinder.007.dae" scale="1.00000 1.00000 1.00000"/>
         </geometry>
       </visual>
@@ -168,5 +168,5 @@
         <origin rpy="0.01967 0.01541 -0.18756" xyz="0.00000 -0.00000 -0.00000"/>
         <geometry>
-          <mesh filename="$(find rover_kachau)/meshes/dae/Cylinder.004.dae" scale="1.00000 1.00000 1.00000"/>
+          <mesh filename="package://rover_kachau/meshes/dae/Cylinder.004.dae" scale="1.00000 1.00000 1.00000"/>
         </geometry>
       </collision>
@@ -180,5 +180,5 @@
         <origin rpy="-0.00000 -0.00000 0.00000" xyz="0.00000 -0.00000 0.00000"/>
         <geometry>
-          <mesh filename="$(find rover_kachau)/meshes/dae/Cylinder.008.dae" scale="1.00000 1.00000 1.00000"/>
+          <mesh filename="package://rover_kachau/meshes/dae/Cylinder.008.dae" scale="1.00000 1.00000 1.00000"/>
         </geometry>
       </visual>
@@ -208,5 +208,5 @@
         <origin rpy="0.01967 0.01541 -0.18756" xyz="-0.00000 0.00000 -0.00000"/>
         <geometry>
-          <mesh filename="$(find rover_kachau)/meshes/dae/Cylinder.001.dae" scale="1.00000 1.00000 1.00000"/>
+          <mesh filename="package://rover_kachau/meshes/dae/Cylinder.001.dae" scale="1.00000 1.00000 1.00000"/>
         </geometry>
       </collision>
@@ -220,5 +220,5 @@
         <origin rpy="-0.00000 0.00000 0.00000" xyz="-0.00000 0.00000 -0.00000"/>
         <geometry>
-          <mesh filename="$(find rover_kachau)/meshes/dae/Cylinder.005.dae" scale="1.00000 1.00000 1.00000"/>
+          <mesh filename="package://rover_kachau/meshes/dae/Cylinder.005.dae" scale="1.00000 1.00000 1.00000"/>
         </geometry>
       </visual>
@@ -248,5 +248,5 @@
         <origin rpy="0.01967 0.01541 -0.18756" xyz="0.00000 0.00000 -0.00000"/>
         <geometry>
-          <mesh filename="$(find rover_kachau)/meshes/dae/Cylinder.003.dae" scale="1.00000 1.00000 1.00000"/>
+          <mesh filename="package://rover_kachau/meshes/dae/Cylinder.003.dae" scale="1.00000 1.00000 1.00000"/>
         </geometry>
       </collision>
@@ -260,5 +260,5 @@
         <origin rpy="-0.00000 0.00000 0.00000" xyz="0.00000 0.00000 0.00000"/>
         <geometry>
-          <mesh filename="$(find rover_kachau)/meshes/dae/Cylinder.006.dae" scale="1.00000 1.00000 1.00000"/>
+          <mesh filename="package://rover_kachau/meshes/dae/Cylinder.006.dae" scale="1.00000 1.00000 1.00000"/>
         </geometry>
       </visual>

Commit message: comunicado oficial: la herramienta está en su sitio con los ejes correctos y todo, gracias gracias me ha costado

File: practica3/rover_kachau/robots/robot.urdf.xacro (robot description, xacro)
@@ -28,4 +28,5 @@
 <!-- Arm -->
 <xacro:scara prefix="" parent_link="base_link"/>
+<xacro:gripper prefix="" parent_link="_rot_link4_link"/>
 <!--
 <xacro:include filename="$(find rover_kachau)/urdf/ros2_control.urdf.xacro"/>

File: practica3/rover_kachau/urdf/arm/gripper.urdf.xacro (robot description, xacro)
@@ -2,33 +2,28 @@
 <robot xmlns:xacro="http://www.ros.org/wiki/xacro">
   <xacro:macro name="gripper" params="prefix parent_link">
-    <joint name="${prefix}_gripper_mount_joint" type="fixed">
+    <joint name="${prefix}_pris_link4_link_joint" type="prismatic">
+      <limit lower="-0.130" upper="2" effort="0.00000" velocity="0.00000"/>
+      <origin rpy="3.14159 0 -1.5708" xyz="0 0 0"/>
       <parent link="${parent_link}"/>
       <child link="${prefix}_pris_link4_link"/>
-      <origin xyz="0 0 0" rpy="3.14159 0 0"/>
-    </joint>
-    <joint name="${prefix}_pris_link4_link_joint" type="prismatic">
-      <limit lower="-0.20000" upper="2.30000" effort="0.00000" velocity="0.00000"/>
-      <origin rpy="3.14159 -0.00000 1.57080" xyz="-0.00000 -0.00000 -0.00000"/>
-      <parent link="${prefix}_rot_link4_link"/>
-      <child link="${prefix}_pris_link4_link"/>
-      <axis xyz="0.00000 0.00000 1.00000"/>
+      <axis xyz="0 0 1"/>
     </joint>
     <joint name="${prefix}_pris_link4.001_link_joint" type="prismatic">
       <limit lower="0.00000" upper="0.20000" effort="0.00000" velocity="0.00000"/>
-      <origin rpy="-3.14159 -1.57080 3.14159" xyz="0.34912 0.00059 0.07033"/>
+      <origin rpy="0 0 3.14159" xyz="0.34568 0.00059 0.07033"/>
       <parent link="${prefix}_pris_link4_link"/>
       <child link="${prefix}_pris_link4.001_link"/>
-      <axis xyz="0.00000 0.00000 1.00000"/>
+      <axis xyz="0 0 1"/>
     </joint>
     <joint name="${prefix}_pris_link4.002_link_joint" type="prismatic">
       <limit lower="0.00000" upper="0.20000" effort="0.00000" velocity="0.00000"/>
-      <origin rpy="-0.00000 1.57080 0.00000" xyz="-0.34568 0.00059 0.07033"/>
+      <origin rpy="3.14159 3.14159 -3.14159" xyz="-0.34568 0.00059 0.07033"/>
       <parent link="${prefix}_pris_link4_link"/>
       <child link="${prefix}_pris_link4.002_link"/>
-      <axis xyz="0.00000 0.00000 1.00000"/>
+      <axis xyz="0 0 1"/>
     </joint>
     <link name="${prefix}_pris_link4_link">
       <collision name="pris_link4_collision">
-        <origin rpy="3.14159 0.00000 -3.14159" xyz="-0.00000 0.00000 -0.00000"/>
+        <origin rpy="-3.14159 0 0" xyz="0 0 0"/>
         <geometry>
           <mesh filename="package://rover_kachau/meshes/dae/Cylinder.013.dae" scale="0.03922 0.03922 0.61477"/>
@@ -37,10 +32,10 @@
       <inertial>
         <inertia ixx="0.00071" ixy="0.00000" ixz="-0.00000" iyy="0.00072" iyz="0.00000" izz="0.00001"/>
-        <origin rpy="0.00000 0.00000 0.00000" xyz="-0.00000 0.00000 0.00000"/>
+        <origin rpy="0 0 0" xyz="0 0 0"/>
         <mass value="0.00100"/>
       </inertial>
       <visual name="pris_link4">
         <material name="Material.004"/>
-        <origin rpy="3.14159 0.00000 3.14159" xyz="-0.00000 0.00000 -0.00000"/>
+        <origin rpy="-3.14159 0 0" xyz="0 0 0"/>
         <geometry>
           <mesh filename="package://rover_kachau/meshes/dae/Cylinder.013.dae" scale="0.03922 0.03922 0.61477"/>
@@ -50,5 +45,5 @@
     <link name="${prefix}_pris_link4.001_link">
       <collision name="pris_link4.001_collision">
-        <origin rpy="0.00000 -1.57080 0.00000" xyz="-0.00000 -0.00000 -0.00000"/>
+        <origin rpy="0 0 0" xyz="0 0 0"/>
         <geometry>
           <box size="0.02510 0.06000 0.09410"/>
@@ -57,10 +52,10 @@
       <inertial>
         <inertia ixx="0.00052" ixy="0.00000" ixz="0.00000" iyy="0.00040" iyz="0.00000" izz="0.00018"/>
-        <origin rpy="0.00000 0.00000 0.00000" xyz="-0.00000 0.00000 0.00000"/>
+        <origin rpy="0 0 0" xyz="0 0 0"/>
         <mass value="0.50000"/>
       </inertial>
       <visual name="pris_link4.001">
         <material name="Material.003"/>
-        <origin rpy="-0.00000 -1.57080 0.00000" xyz="-0.00000 -0.00000 -0.00000"/>
+        <origin rpy="0 0 0" xyz="0 0 0"/>
         <geometry>
           <mesh filename="package://rover_kachau/meshes/dae/Cylinder.009.dae" scale="0.03922 0.03922 0.61477"/>
@@ -70,5 +65,5 @@
     <link name="${prefix}_pris_link4.002_link">
       <collision name="pris_link4.002_collision">
-        <origin rpy="-3.14159 -1.57080 -3.14159" xyz="0.00000 0.00000 -0.00000"/>
+        <origin rpy="-3.14159 -3.14159 0" xyz="0 0 0"/>
         <geometry>
           <box size="0.02510 0.06000 0.09410"/>
@@ -77,10 +72,10 @@
       <inertial>
         <inertia ixx="0.00052" ixy="-0.00000" ixz="0.00000" iyy="0.00040" iyz="-0.00000" izz="0.00018"/>
-        <origin rpy="0.00000 0.00000 0.00000" xyz="0.00000 0.00000 -0.00000"/>
-        <mass value="0.50000"/>
+        <origin rpy="0 0 0" xyz="0 0 0"/>
+        <mass value="0.00100"/>
       </inertial>
       <visual name="pris_link4.002">
         <material name="Material.004"/>
-        <origin rpy="0.00000 1.57080 0.00000" xyz="0.00000 0.00000 -0.00000"/>
+        <origin rpy="0 0 3.14159" xyz="0 0 0"/>
         <geometry>
           <mesh filename="package://rover_kachau/meshes/dae/Cylinder.010.dae" scale="0.03922 0.03922 0.61477"/>

File: practica3/rover_kachau/urdf/arm/scara.urdf.xacro (robot description, xacro)
@@ -32,11 +32,4 @@
       <parent link="${prefix}_link3_link"/>
       <child link="${prefix}_rot_link4_link"/>
-      <axis xyz="0.00000 0.00000 1.00000"/>
-    </joint>
-    <joint name="${prefix}_pris_link4_link_joint" type="prismatic">
-      <limit lower="-0.5" upper="0.5" effort="0.00000" velocity="0.00000"/>
-      <origin rpy="0.00000 0.00000 0.00000" xyz="0.00000 0.00000 0.00000"/>
-      <parent link="${prefix}_rot_link4_link"/>
-      <child link="${prefix}_pris_link4_link"/>
       <axis xyz="0.00000 0.00000 1.00000"/>
     </joint>
@@ -141,24 +134,4 @@
       </visual>
     </link>
-    <link name="${prefix}_pris_link4_link">
-      <collision name="pris_link4_collision">
-        <origin rpy="3.14159 0.00000 -3.14159" xyz="-0.00000 0.00000 -0.00000"/>
-        <geometry>
-          <mesh filename="package://rover_kachau/meshes/dae/Cylinder.013.dae" scale="0.03922 0.03922 0.61477"/>
-        </geometry>
-      </collision>
-      <inertial>
-        <inertia ixx="0.00071" ixy="0.00000" ixz="-0.00000" iyy="0.00072" iyz="0.00000" izz="0.00001"/>
-        <origin rpy="0.00000 0.00000 0.00000" xyz="-0.00000 0.00000 0.00000"/>
-        <mass value="0.00100"/>
-      </inertial>
-      <visual name="pris_link4">
-        <material name="Material.004"/>
-        <origin rpy="3.14159 0.00000 3.14159" xyz="-0.00000 0.00000 -0.00000"/>
-        <geometry>
-          <mesh filename="package://rover_kachau/meshes/dae/Cylinder.013.dae" scale="0.03922 0.03922 0.61477"/>
-        </geometry>
-      </visual>
-    </link>
   </xacro:macro>
 </robot>

File: practica3/rover_kachau/urdf/base/robot_base.urdf.xacro (robot description, xacro)
@@ -49,7 +49,5 @@
           <mesh filename="package://rover_kachau/meshes/dae/Cube.001.dae" scale="1.0 1.0 1.0"/>
         </geometry>
-        <material name="chassis_mat">
-          <color rgba="0.5 0.5 0.5 1"/>
-        </material>
+        <material name="Material.004"/>
       </visual>
     </link>
