Commit message: uf OOF

File: practica3/rover_kachau/robots/robot.urdf.xacro (robot description, xacro)
@@ -29,7 +29,5 @@
 <xacro:scara prefix="" parent_link="base_link"/>
 <xacro:gripper prefix="" parent_link="_rot_link4_link"/>
-<!--
 <xacro:include filename="$(find rover_kachau)/urdf/ros2_control.urdf.xacro"/>
 <xacro:arg name="config_controllers" default="$(find rover_kachau)/config/rover_controllers.yaml"/>
--->
 </robot>

File: practica3/rover_kachau/urdf/sensors/camera.urdf.xacro (robot description, xacro)
@@ -1,34 +1,98 @@
 <?xml version="1.0"?>
 <robot xmlns:xacro="http://www.ros.org/wiki/xacro">
-  <xacro:macro name="camera_sensor" params="frame_prefix parent_link horizontal_fov video_width video_height">
-    <link name="${frame_prefix}_camera_link"/>
-    <joint name="${frame_prefix}_camera_joint" type="fixed">
+<xacro:macro name="camera_sensor"
+  params="frame_prefix
+          parent_link
+          *origin
+          node_name:=camera
+          node_namespace:=${None}
+          topic_prefix:=~/
+          horizontal_fov:=80
+          vertical_fov:=60
+          video_width:=1280
+          video_height:=720
+          video_fps:=30">
+  <xacro:if value="${node_namespace == None}">
+    <xacro:property name="node_namespace" value="${node_name}"/>
+  </xacro:if>
+  <!-- Camera base link -->
+  <joint name="${frame_prefix}_camera_base_joint" type="fixed">
+    <xacro:insert_block name="origin"/>
+    <parent link="${parent_link}"/>
+    <child link="${frame_prefix}_camera_base_link"/>
+  </joint>
+  <link name="${frame_prefix}_camera_base_link">
+    <visual>
+      <origin xyz="0 0 0" rpy="0 0 0"/>
+      <geometry>
+        <box size="0.025 0.05 0.025"/>
+      </geometry>
+      <material name="light_grey">
+        <color rgba="0.35 0.35 0.35 1"/>
+      </material>
+    </visual>
+    <collision>
+      <origin xyz="0.0 0.0 0.0" rpy="0 0 0"/>
+      <geometry>
+        <box size="0.025 0.05 0.025"/>
+      </geometry>
+    </collision>
+    <inertial>
+      <mass value="0.135"/>
+      <origin xyz="0 0 0"/>
+      <xacro:solid_cuboid_inertia m="0.135" w="0.033" h="0.175" d="0.03"/>
+    </inertial>
+  </link>
+  <!-- Camera optical frame -->
+  <joint name="${frame_prefix}_camera_joint" type="fixed">
+    <origin xyz="0.0 -0.06 0.0" rpy="0.0 0.0 0.0"/>
+    <parent link="${frame_prefix}_camera_base_link"/>
+    <child link="${frame_prefix}_camera_frame"/>
+  </joint>
+  <link name="${frame_prefix}_camera_frame"/>
+  <joint name="${frame_prefix}color_optical_joint" type="fixed">
+    <origin xyz="0.0 0.0 0.0" rpy="${-pi/2} 0.0 ${-pi/2}"/>
+    <parent link="${frame_prefix}_camera_frame"/>
+    <child link="${frame_prefix}_camera_optical_frame"/>
+  </joint>
+  <link name="${frame_prefix}_camera_optical_frame"/>
+  <gazebo reference="${frame_prefix}_camera_frame">
+    <sensor name="${frame_prefix}_sensor" type="camera">
+      <visualize>true</visualize>
+      <update_rate>${video_fps}</update_rate>
+      <topic>/${frame_prefix}/image</topic>
+      <camera>
+        <horizontal_fov>${horizontal_fov}</horizontal_fov>
+        <image>
+          <width>${video_width}</width>
+          <height>${video_height}</height>
+          <format>R8G8B8</format>
+        </image>
+        <clip>
+          <near>0.10</near>
+          <far>15.0</far>
+        </clip>
+        <noise>
+          <type>gaussian</type>
+          <mean>0.0</mean>
+          <stddev>0.007</stddev>
+        </noise>
+        <optical_frame_id>${frame_prefix}_camera_optical_frame</optical_frame_id>
+      </camera>
+    </sensor>
+  </gazebo>
+</xacro:macro>
+  <xacro:macro name="imu_sensor" params="prefix topic parent_link">
+    <link name="${prefix}_imu_link"/>
+    <joint name="${prefix}_imu_joint" type="fixed">
       <parent link="${parent_link}"/>
-      <child link="${frame_prefix}_camera_link"/>
+      <child link="${prefix}_imu_link"/>
       <origin xyz="0 0 0" rpy="0 0 0"/>
     </joint>
-    <gazebo reference="${frame_prefix}_camera_link">
-      <sensor name="${frame_prefix}_sensor" type="camera">
-        <visualize>true</visualize>
+    <gazebo reference="${prefix}_imu_link">
+      <sensor name="${prefix}_sensor" type="imu">
+        <always_on>1</always_on>
         <update_rate>30</update_rate>
-        <topic>/${frame_prefix}/image</topic>
-        <camera>
-          <horizontal_fov>${horizontal_fov}</horizontal_fov>
-          <image>
-            <width>${video_width}</width>
-            <height>${video_height}</height>
-            <format>R8G8B8</format>
-          </image>
-          <clip>
-            <near>0.10</near>
-            <far>15.0</far>
-          </clip>
-          <noise>
-            <type>gaussian</type>
-            <mean>0.0</mean>
-            <stddev>0.007</stddev>
-          </noise>
-          <optical_frame_id>${frame_prefix}_camera_link</optical_frame_id>
-        </camera>
+        <topic>${topic}</topic>
       </sensor>
     </gazebo>

File: practica3/rover_kachau/urdf/sensors/gps.urdf.xacro (robot description, xacro)
@@ -1,19 +1,48 @@
 <?xml version="1.0"?>
 <robot xmlns:xacro="http://www.ros.org/wiki/xacro">
-  <xacro:macro name="gps_sensor" params="frame_prefix update_rate parent_link">
-    <link name="${frame_prefix}_gps_link"/>
-    <joint name="${frame_prefix}_gps_joint" type="fixed">
-      <parent link="${parent_link}"/>
-      <child link="${frame_prefix}_gps_link"/>
-      <origin xyz="0 0 0" rpy="0 0 0"/>
-    </joint>
-    <gazebo reference="${frame_prefix}_gps_link">
-      <sensor name="${frame_prefix}_sensor" type="navsat">
-        <always_on>1</always_on>
-        <update_rate>${update_rate}</update_rate>
-        <topic>/robot/gps/fix</topic>
-        <gz_frame_id>${frame_prefix}_gps_link</gz_frame_id>
-      </sensor>
-    </gazebo>
-  </xacro:macro>
+<xacro:macro name="sensor_gps"
+  params="frame_prefix
+          parent
+          *origin
+          simulation:=false
+          node_name:=gps
+          node_namespace:=${None}
+          topic_prefix:=~/
+          update_rate:=5.0">
+  <joint name="${frame_prefix}_joint" type="fixed">
+    <xacro:insert_block name="origin"/>
+    <parent link="${parent}"/>
+    <child link="${frame_prefix}_base_link"/>
+  </joint>
+  <link name="${frame_prefix}_base_link">
+    <inertial>
+      <origin xyz="0.0 0.0 0.015" rpy="0 0 0"/>
+      <mass value="0.2"/>
+      <xacro:solid_cuboid_inertia m="0.2" w="0.081" h="0.081" d="0.03"/>
+    </inertial>
+    <visual>
+      <origin rpy="0 0 0" xyz="0 0 0"/>
+      <material name="gps_color">
+        <color rgba="1 1 1 1"/>
+      </material>
+      <geometry>
+        <box size="0.075 0.075 0.025"/>
+      </geometry>
+    </visual>
+    <collision>
+      <origin rpy="0 0 0" xyz="0 0 0"/>
+      <geometry>
+        <box size="0.075 0.075 0.025"/>
+      </geometry>
+    </collision>
+  </link>
+  <gazebo reference="${frame_prefix}_base_link">
+    <sensor name="${frame_prefix}_sensor" type="navsat">
+      <always_on>1</always_on>
+      <update_rate>${update_rate}</update_rate>
+      <topic>/robot/gps/fix</topic>
+      <gz_frame_id>${frame_prefix}_base_link</gz_frame_id>
+    </sensor>
+  </gazebo>
+</xacro:macro>
 </robot>

File: practica3/rover_kachau/urdf/sensors/gpu_lidar.urdf.xacro (robot description, xacro)
@@ -1,41 +1,75 @@
 <?xml version="1.0"?>
 <robot xmlns:xacro="http://www.ros.org/wiki/xacro">
-  <xacro:macro name="lidar_sensor" params="frame_prefix parent_link topic">
-    <link name="${frame_prefix}_lidar_link"/>
-    <joint name="${frame_prefix}_lidar_joint" type="fixed">
-      <parent link="${parent_link}"/>
-      <child link="${frame_prefix}_lidar_link"/>
+<xacro:macro name="sensor_3d_lidar"
+  params="frame_prefix
+          parent
+          *origin
+          node_name:=sensor_3d_lidar
+          node_namespace:=${None}
+          topic_prefix:=~/
+          gpu:=true">
+  <joint name="${frame_prefix}_base_joint" type="fixed">
+    <xacro:insert_block name="origin"/>
+    <parent link="${parent}"/>
+    <child link="${frame_prefix}_base_link"/>
+  </joint>
+  <link name="${frame_prefix}_base_link">
+    <collision>
       <origin xyz="0 0 0" rpy="0 0 0"/>
-    </joint>
-    <gazebo reference="${frame_prefix}_lidar_link">
-      <sensor name="gpu_lidar" type="gpu_lidar">
-        <pose relative_to="${frame_prefix}_lidar_link">0 0 0 0 0 0</pose>
-        <topic>${topic}</topic>
-        <update_rate>20</update_rate>
-        <gz_frame_id>${frame_prefix}_lidar_link</gz_frame_id>
-        <lidar>
-          <scan>
-            <horizontal>
-              <samples>450</samples>
-              <resolution>1</resolution>
-              <min_angle>-3.141592</min_angle>
-              <max_angle>3.141592</max_angle>
-            </horizontal>
-            <vertical>
-              <samples>32</samples>
-              <resolution>1</resolution>
-              <min_angle>-0.436332</min_angle>
-              <max_angle>0.08726</max_angle>
-            </vertical>
-          </scan>
-          <range>
-            <min>0.2</min>
-            <max>90.0</max>
-            <resolution>0.02</resolution>
-          </range>
-        </lidar>
-        <visualize>true</visualize>
-      </sensor>
-    </gazebo>
-  </xacro:macro>
+      <geometry>
+        <cylinder radius="0.05" length="0.1"/>
+      </geometry>
+    </collision>
+    <visual>
+      <origin xyz="0 0 0" rpy="0 0 0"/>
+      <geometry>
+        <cylinder radius="0.05" length="0.1"/>
+      </geometry>
+      <material name="blackgray_color">
+        <color rgba="0.25 0.25 0.25 1"/>
+      </material>
+    </visual>
+    <inertial>
+      <mass value="1.0"/>
+      <origin xyz="0 0 0.04135"/>
+      <xacro:solid_cylinder_inertia m="1.0" r="0.05" h="0.1"/>
+    </inertial>
+  </link>
+  <joint name="${frame_prefix}_joint" type="fixed">
+    <parent link="${frame_prefix}_base_link"/>
+    <child link="${frame_prefix}_link"/>
+    <origin xyz="0.0 0.0 0.0635" rpy="0 0 0"/>
+  </joint>
+  <link name="${frame_prefix}_link"/>
+  <gazebo reference="${frame_prefix}_link">
+    <sensor name="gpu_lidar" type="gpu_lidar">
+      <pose relative_to="${frame_prefix}_link">0 0 0 0 0 0</pose>
+      <topic>${frame_prefix}_sensor</topic>
+      <update_rate>20</update_rate>
+      <gz_frame_id>${frame_prefix}_link</gz_frame_id>
+      <lidar>
+        <scan>
+          <horizontal>
+            <samples>450</samples>
+            <resolution>1</resolution>
+            <min_angle>-3.141592</min_angle>
+            <max_angle>3.141592</max_angle>
+          </horizontal>
+          <vertical>
+            <samples>32</samples>
+            <resolution>1</resolution>
+            <min_angle>-0.436332</min_angle>
+            <max_angle>0.08726</max_angle>
+          </vertical>
+        </scan>
+        <range>
+          <min>0.2</min>
+          <max>90.0</max>
+          <resolution>0.02</resolution>
+        </range>
+      </lidar>
+      <visualize>true</visualize>
+    </sensor>
+  </gazebo>
+</xacro:macro>
 </robot>

File: practica3/rover_kachau/urdf/sensors/imu_sensor.urdf.xacro (robot description, xacro)
@@ -1,18 +1,31 @@
 <?xml version="1.0"?>
 <robot xmlns:xacro="http://www.ros.org/wiki/xacro">
-  <xacro:macro name="imu_sensor" params="prefix topic parent_link">
-    <link name="${prefix}_imu_link"/>
-    <joint name="${prefix}_imu_joint" type="fixed">
-      <parent link="${parent_link}"/>
-      <child link="${prefix}_imu_link"/>
-      <origin xyz="0 0 0" rpy="0 0 0"/>
-    </joint>
-    <gazebo reference="${prefix}_imu_link">
-      <sensor name="${prefix}_sensor" type="imu">
-        <always_on>1</always_on>
-        <update_rate>30</update_rate>
-        <topic>${topic}</topic>
-      </sensor>
-    </gazebo>
-  </xacro:macro>
+<xacro:macro name="sensor_imu" params="prefix ns:='' topic:='imu/data' parent *origin">
+  <joint name="${prefix}_joint" type="fixed">
+    <axis xyz="1 0 0"/>
+    <xacro:insert_block name="origin"/>
+    <parent link="${parent}"/>
+    <child link="${prefix}_link"/>
+  </joint>
+  <link name="${prefix}_link">
+    <inertial>
+      <origin xyz="0.0 0.0 0.01" rpy="0 0 0"/>
+      <mass value="0.005"/>
+      <xacro:solid_cuboid_inertia m="0.005" w="0.001" h="0.001" d="0.001"/>
+    </inertial>
+    <visual>
+      <origin rpy="0 0 0" xyz="0 0 0"/>
+      <geometry>
+        <box size="0.001 0.001 0.001"/>
+      </geometry>
+    </visual>
+  </link>
+  <gazebo reference="${prefix}_link">
+    <sensor name="${prefix}_sensor" type="imu">
+      <always_on>1</always_on>
+      <update_rate>30</update_rate>
+      <topic>${topic}</topic>
+    </sensor>
+  </gazebo>
+</xacro:macro>
 </robot>

File: practica3/rover_kachau/urdf/sensors/sensors.urdf.xacro (robot description, xacro)
@@ -5,5 +5,7 @@
   <xacro:include filename="$(find rover_kachau)/urdf/sensors/gpu_lidar.urdf.xacro"/>
   <xacro:include filename="$(find rover_kachau)/urdf/sensors/gps.urdf.xacro"/>
-  <xacro:imu_sensor prefix="imu" topic="/imu/data" parent_link="base_link"/>
+  <xacro:sensor_imu prefix="imu" parent="base_link">
+    <origin xyz="0 0 0.1" rpy="0 0 0"/>
+  </xacro:sensor_imu>
   <xacro:camera_sensor
     frame_prefix="front_cam"
@@ -11,6 +13,12 @@
     horizontal_fov="1.57"
     video_width="640"
-    video_height="480"/>
-  <xacro:lidar_sensor frame_prefix="lidar" parent_link="base_link" topic="/lidar/scan"/>
-  <xacro:gps_sensor frame_prefix="gps" update_rate="10" parent_link="base_link"/>
+    video_height="480">
+    <origin xyz="0.5 0 0.3" rpy="0 0 0"/>
+  </xacro:camera_sensor>
+  <xacro:sensor_3d_lidar frame_prefix="lidar" parent="base_link">
+    <origin xyz="0 0 0.3" rpy="0 0 0"/>
+  </xacro:sensor_3d_lidar>
+  <xacro:sensor_gps frame_prefix="gps" parent="base_link">
+    <origin xyz="0 0 0.2" rpy="0 0 0"/>
+  </xacro:sensor_gps>
 </robot>

Commit message: faltaban cerrar slip1 slip2, un typo etc. asistente responde

File: practica3/rover_kachau/robots/robot.urdf.xacro (robot description, xacro)
@@ -1,12 +1,8 @@
 <?xml version="1.0"?>
 <robot name="robot" xmlns:xacro="http://www.ros.org/wiki/xacro">
-<!-- includes -->
-<xacro:include filename="$(find rover_kachau)/urdf/base/robot_base.urdf.xacro"/>
-<xacro:include filename="$(find rover_kachau)/urdf/wheels/rover_wheel.urdf.xacro"/>
-<xacro:include filename="$(find rover_kachau)/urdf/arm/gripper.urdf.xacro"/>
-<xacro:include filename="$(find rover_kachau)/urdf/arm/scara.urdf.xacro"/>
-<xacro:include filename="$(find rover_kachau)/urdf/sensors/sensors.urdf.xacro"/>
-<xacro:include filename="$(find rover_kachau)/urdf/tank/rover_tank.urdf.xacro"/>
-<xacro:include filename="$(find rover_kachau)/urdf/utils/utils.urdf.xacro"/>
+<!-- argumentos -->
+<xacro:arg name="robot_ns" default=""/>
+<xacro:arg name="prefix" default=""/>
+<xacro:arg name="config_controllers" default="$(find rover_kachau)/config/rover_controllers.yaml"/>
 <!-- Propiedades -->
 <xacro:property name="PI" value="3.1415926535897931"/>
@@ -17,7 +13,13 @@
 <xacro:property name="arm_offset_y" value="0.82"/>
 <xacro:property name="arm_offset_z" value="0.69"/>
-<!-- argumentos -->
-<xacro:arg name="robot_ns" default=""/>
-<xacro:arg name="prefix" default=""/>
+<!-- includes -->
+<xacro:include filename="$(find rover_kachau)/urdf/utils/utils.urdf.xacro"/>
+<xacro:include filename="$(find rover_kachau)/urdf/base/robot_base.urdf.xacro"/>
+<xacro:include filename="$(find rover_kachau)/urdf/wheels/rover_wheel.urdf.xacro"/>
+<xacro:include filename="$(find rover_kachau)/urdf/arm/gripper.urdf.xacro"/>
+<xacro:include filename="$(find rover_kachau)/urdf/arm/scara.urdf.xacro"/>
+<xacro:include filename="$(find rover_kachau)/urdf/sensors/sensors.urdf.xacro"/>
+<xacro:include filename="$(find rover_kachau)/urdf/tank/rover_tank.urdf.xacro"/>
+<xacro:include filename="$(find rover_kachau)/urdf/ros2_control.urdf.xacro"/>
 <!-- Base -->
 <xacro:robot_base prefix="$(arg prefix)"/>
@@ -29,5 +31,3 @@
 <xacro:scara prefix="" parent_link="base_link"/>
 <xacro:gripper prefix="" parent_link="_rot_link4_link"/>
-<xacro:include filename="$(find rover_kachau)/urdf/ros2_control.urdf.xacro"/>
-<xacro:arg name="config_controllers" default="$(find rover_kachau)/config/rover_controllers.yaml"/>
 </robot>

File: practica3/rover_kachau/urdf/utils/utils.urdf.xacro (robot description, xacro)
@@ -22,3 +22,13 @@
   <material name="Material.020"><color rgba="0 0 0 1"/></material>
   <material name="Material.021"><color rgba="0 0 0 1"/></material>
+  <xacro:macro name="solid_cuboid_inertia" params="m w h d">
+    <inertia ixx="${(m/12.0) * (h*h + d*d)}" ixy="0" ixz="0"
+             iyy="${(m/12.0) * (w*w + d*d)}" iyz="0"
+             izz="${(m/12.0) * (w*w + h*h)}"/>
+  </xacro:macro>
+  <xacro:macro name="solid_cylinder_inertia" params="m r h">
+    <inertia ixx="${(m/12.0) * (3*r*r + h*h)}" ixy="0" ixz="0"
+             iyy="${(m/12.0) * (3*r*r + h*h)}" iyz="0"
+             izz="${(m*r*r)/2.0}"/>
+  </xacro:macro>
 </robot>

File: practica3/rover_kachau/urdf/wheels/rover_wheel.urdf.xacro (robot description, xacro)
@@ -136,6 +136,6 @@
               <mu2>1.000000</mu2>
               <fdir1>0.000000 0.000000 1.000000</fdir1>
-              <slip1>0.50000<slip1>
-              <slip2>0.50000<slip2>
+              <slip1>0.50000</slip1>
+              <slip2>0.50000</slip2>
             </ode>
           </friction>
@@ -187,6 +187,6 @@
               <mu2>1.000000</mu2>
               <fdir1>0.000000 0.000000 1.000000</fdir1>
-              <slip1>0.50000<slip1>
-              <slip2>0.50000<slip2>
+              <slip1>0.50000</slip1>
+              <slip2>0.50000</slip2>
             </ode>
           </friction>
@@ -238,6 +238,6 @@
               <mu2>1.000000</mu2>
               <fdir1>0.000000 0.000000 1.000000</fdir1>
-              <slip1>0.50000<slip1>
-              <slip2>0.50000<slip2>
+              <slip1>0.50000</slip1>
+              <slip2>0.50000</slip2>
             </ode>
           </friction>
@@ -289,6 +289,6 @@
               <mu2>1.000000</mu2>
               <fdir1>0.000000 0.000000 1.000000</fdir1>
-              <slip1>0.50000<slip1>
-              <slip2>0.50000<slip2>
+              <slip1>0.50000</slip1>
+              <slip2>0.50000</slip2>
             </ode>
           </friction>
