Commit message: smt wrong with controllers launch. gitignore for repo world

File: practica3/robot_moveit_config/config/robot.ros2_control.xacro (robot description, xacro)
@@ -6,5 +6,5 @@
             <hardware>
                 <!-- By default, set up controllers for simulation. This won't work on real hardware -->
-                <plugin>mock_components/GenericSystem</plugin>
+                <plugin>gz_ros2_control/GazeboSimSystem</plugin>
             </hardware>
             <joint name="_link2_link_joint">

File: practica3/robot_moveit_config/config/robot.urdf.xacro (robot description, xacro)
@@ -4,4 +4,5 @@
     <!-- Import robot urdf file -->
     <xacro:include filename="$(find rover_kachau)/robots/robot.urdf.xacro" />
+    <xacro:include filename="robot.srdf" />
     <!-- Import control_xacro -->
     <xacro:include filename="robot.ros2_control.xacro" />

File: practica3/rover_kachau/urdf/arm/gripper.urdf.xacro (robot description, xacro)
@@ -11,5 +11,5 @@
     <joint name="${prefix}_pris_link4.001_link_joint" type="prismatic">
       <limit lower="0.00000" upper="0.20000" effort="0.00000" velocity="0.00000"/>
-      <origin rpy="0 0 3.14159" xyz="0.34568 0.00059 0.07033"/>
+      <origin rpy="0 1.5708 3.14159" xyz="0.34568 0.00059 0.07033"/>
       <parent link="${prefix}_pris_link4_link"/>
       <child link="${prefix}_pris_link4.001_link"/>
@@ -18,5 +18,5 @@
     <joint name="${prefix}_pris_link4.002_link_joint" type="prismatic">
       <limit lower="0.00000" upper="0.20000" effort="0.00000" velocity="0.00000"/>
-      <origin rpy="3.14159 3.14159 -3.14159" xyz="-0.34568 0.00059 0.07033"/>
+      <origin rpy="3.14159 1.5708 -3.14159" xyz="-0.34568 0.00059 0.07033"/>
       <parent link="${prefix}_pris_link4_link"/>
       <child link="${prefix}_pris_link4.002_link"/>
@@ -57,5 +57,5 @@
       <visual name="pris_link4.001">
         <material name="Material.003"/>
-        <origin rpy="0 0 0" xyz="0 0 0"/>
+        <origin rpy="0 -1.5708 0" xyz="0 0 0"/>
         <geometry>
           <mesh filename="package://rover_kachau/meshes/dae/Cylinder.009.dae" scale="0.03922 0.03922 0.61477"/>
@@ -65,5 +65,5 @@
     <link name="${prefix}_pris_link4.002_link">
       <collision name="pris_link4.002_collision">
-        <origin rpy="-3.14159 -3.14159 0" xyz="0 0 0"/>
+        <origin rpy="0 -1.5708 3.14159" xyz="0 0 0"/>
         <geometry>
           <box size="0.02510 0.06000 0.09410"/>
@@ -77,5 +77,5 @@
       <visual name="pris_link4.002">
         <material name="Material.004"/>
-        <origin rpy="0 0 3.14159" xyz="0 0 0"/>
+        <origin rpy="0 -1.5708 3.14159" xyz="0 0 0"/>
         <geometry>
           <mesh filename="package://rover_kachau/meshes/dae/Cylinder.010.dae" scale="0.03922 0.03922 0.61477"/>
