Commit message: the rover didnt move cause i hadnt add the limits for effort and speed was set to 0. changes on urdf do not affect moveit previous configuration

File: practica3/src/rover_kachau/urdf/arm/gripper.urdf.xacro (robot description, xacro)
@@ -3,5 +3,5 @@
   <xacro:macro name="gripper" params="prefix parent_link">
     <joint name="${prefix}_pris_link4_link_joint" type="prismatic">
-      <limit lower="-0.130" upper="2" effort="0.00000" velocity="0.00000"/>
+      <limit lower="-0.130" upper="2" effort="10.0" velocity="10.0"/>
       <origin rpy="3.14159 0 -1.5708" xyz="0 0 0"/>
       <parent link="${parent_link}"/>
@@ -10,5 +10,5 @@
     </joint>
     <joint name="${prefix}_pris_link4.001_link_joint" type="prismatic">
-      <limit lower="0.00000" upper="0.20000" effort="0.00000" velocity="0.00000"/>
+      <limit lower="0.00000" upper="0.20000" effort="10.0" velocity="10.0"/>
       <origin rpy="0 1.5708 3.14159" xyz="0.34568 0.00059 0.07033"/>
       <parent link="${prefix}_pris_link4_link"/>
@@ -17,5 +17,5 @@
     </joint>
     <joint name="${prefix}_pris_link4.002_link_joint" type="prismatic">
-      <limit lower="0.00000" upper="0.20000" effort="0.00000" velocity="0.00000"/>
+      <limit lower="0.00000" upper="0.20000" effort="10.0" velocity="10.0"/>
       <origin rpy="3.14159 1.5708 -3.14159" xyz="-0.34568 0.00059 0.07033"/>
       <parent link="${prefix}_pris_link4_link"/>

File: practica3/src/rover_kachau/urdf/arm/scara.urdf.xacro (robot description, xacro)
@@ -14,5 +14,5 @@
     </joint>
     <joint name="${prefix}_link2_link_joint" type="continuous">
-      <limit effort="0.00000" velocity="0.00000"/>
+      <limit effort="10.0" velocity="10.0"/>
       <origin rpy="-0.00000 -0.00000 0.00000" xyz="0.00000 -0.00000 0.00000"/>
       <parent link="${prefix}_link1_link"/>
@@ -21,5 +21,5 @@
     </joint>
     <joint name="${prefix}_link3_link_joint" type="revolute">
-      <limit lower="-3.14000" upper="3.14000" effort="0.00000" velocity="0.00000"/>
+      <limit lower="-3.14000" upper="3.14000" effort="10.0" velocity="10.0"/>
       <origin rpy="0.00000 0.00000 1.57080" xyz="0.96320 -0.00000 0.06102"/>
       <parent link="${prefix}_link2_link"/>
@@ -28,5 +28,5 @@
     </joint>
     <joint name="${prefix}_rot_link4_link_joint" type="continuous">
-      <limit effort="0.00000" velocity="0.00000"/>
+      <limit effort="10.0" velocity="10.0"/>
       <origin rpy="0.00000 0.00000 -0.00000" xyz="-0.99849 0.00559 -0.52727"/>
       <parent link="${prefix}_link3_link"/>

File: practica3/src/rover_kachau/urdf/ros2_control.urdf.xacro (robot description, xacro)
@@ -47,55 +47,4 @@
       <state_interface name="effort"/>
     </joint>
-    <joint name="_link2_link_joint">
-      <command_interface name="position">
-        <param name="min">-3.14</param>
-        <param name="max">3.14</param>
-      </command_interface>
-      <state_interface name="position"/>
-      <state_interface name="velocity"/>
-      <state_interface name="effort"/>
-    </joint>
-    <joint name="_link3_link_joint">
-      <command_interface name="position">
-        <param name="min">-3.14</param>
-        <param name="max">3.14</param>
-      </command_interface>
-      <state_interface name="position"/>
-      <state_interface name="velocity"/>
-      <state_interface name="effort"/>
-    </joint>
-    <joint name="_rot_link4_link_joint">
-      <command_interface name="position"/>
-      <state_interface name="position"/>
-      <state_interface name="velocity"/>
-      <state_interface name="effort"/>
-    </joint>
-    <joint name="_pris_link4_link_joint">
-      <command_interface name="position">
-        <param name="min">-0.5</param>
-        <param name="max">0.105</param>
-      </command_interface>
-      <state_interface name="position"/>
-      <state_interface name="velocity"/>
-      <state_interface name="effort"/>
-    </joint>
-    <joint name="_pris_link4.001_link_joint">
-      <command_interface name="position">
-        <param name="min">0.0</param>
-        <param name="max">0.20</param>
-      </command_interface>
-      <state_interface name="position"/>
-      <state_interface name="velocity"/>
-      <state_interface name="effort"/>
-    </joint>
-    <joint name="_pris_link4.002_link_joint">
-      <command_interface name="position">
-        <param name="min">0.0</param>
-        <param name="max">0.20</param>
-      </command_interface>
-      <state_interface name="position"/>
-      <state_interface name="velocity"/>
-      <state_interface name="effort"/>
-    </joint>
   </ros2_control>
 </xacro:macro>

File: practica3/src/rover_kachau/urdf/wheels/rover_wheel.urdf.xacro (robot description, xacro)
@@ -19,5 +19,5 @@
     </joint>
     <joint name="${prefix}_frontL_link_joint" type="continuous">
-      <limit effort="0.00000" velocity="0.00000"/>
+      <limit effort="1000.0" velocity="100.0"/>
       <origin rpy="1.56418 -0.93639 3.12224" xyz="-0.02187 -0.29773 -0.28847"/>
       <parent link="${prefix}_armFrontL_link"/>
@@ -32,5 +32,5 @@
     </joint>
     <joint name="${prefix}_frontR_link_joint" type="continuous">
-      <limit effort="0.00000" velocity="0.00000"/>
+      <limit effort="1000.0" velocity="100.0"/>
       <origin rpy="1.56418 -0.93639 3.12224" xyz="-0.02187 0.29825 -0.28847"/>
       <parent link="${prefix}_armFrontR_link"/>
@@ -45,5 +45,5 @@
     </joint>
     <joint name="${prefix}_backL_link_joint" type="continuous">
-      <limit effort="0.00000" velocity="0.00000"/>
+      <limit effort="1000.0" velocity="100.0"/>
       <origin rpy="-1.60020 -0.56075 0.01354" xyz="0.02187 -0.29773 -0.28847"/>
       <parent link="${prefix}_armBackL_link"/>
@@ -58,5 +58,5 @@
     </joint>
     <joint name="${prefix}_backR_link_joint" type="continuous">
-      <limit effort="0.00000" velocity="0.00000"/>
+      <limit effort="1000.0" velocity="100.0"/>
       <origin rpy="-1.60020 -0.56075 0.01354" xyz="0.02187 0.29825 -0.28847"/>
       <parent link="${prefix}_armBackR_link"/>

Commit message: velocities fixed, moveitplugin fixed. execution correcto. wheels were upside down, quick-fixed (if i have time i will cleanly fix it). to fix gripper as soon as tutorial charges also my phone isnt working i cant access uni repos

File: practica3/src/rover_kachau/urdf/arm/gripper.urdf.xacro (robot description, xacro)
@@ -4,4 +4,5 @@
     <joint name="${prefix}_pris_link4_link_joint" type="prismatic">
       <limit lower="-0.130" upper="2" effort="10.0" velocity="10.0"/>
+      <dynamics damping="50.0" friction="10.0"/>
       <origin rpy="3.14159 0 -1.5708" xyz="0 0 0"/>
       <parent link="${parent_link}"/>
@@ -11,4 +12,5 @@
     <joint name="${prefix}_pris_link4.001_link_joint" type="prismatic">
       <limit lower="0.00000" upper="0.20000" effort="10.0" velocity="10.0"/>
+      <dynamics damping="10.0" friction="10.0"/>
       <origin rpy="0 1.5708 3.14159" xyz="0.34568 0.00059 0.07033"/>
       <parent link="${prefix}_pris_link4_link"/>
@@ -18,4 +20,5 @@
     <joint name="${prefix}_pris_link4.002_link_joint" type="prismatic">
       <limit lower="0.00000" upper="0.20000" effort="10.0" velocity="10.0"/>
+      <dynamics damping="10.0" friction="10.0"/>
       <origin rpy="3.14159 1.5708 -3.14159" xyz="-0.34568 0.00059 0.07033"/>
       <parent link="${prefix}_pris_link4_link"/>

Commit message: el gripper tenia los limites mal

File: practica3/src/rover_kachau/urdf/arm/gripper.urdf.xacro (robot description, xacro)
@@ -11,5 +11,5 @@
     </joint>
     <joint name="${prefix}_pris_link4.001_link_joint" type="prismatic">
-      <limit lower="0.00000" upper="0.20000" effort="10.0" velocity="10.0"/>
+      <limit lower="0.00000" upper="0.20000" effort="100.0" velocity="1.0"/>
       <dynamics damping="10.0" friction="10.0"/>
       <origin rpy="0 1.5708 3.14159" xyz="0.34568 0.00059 0.07033"/>
@@ -19,5 +19,5 @@
     </joint>
     <joint name="${prefix}_pris_link4.002_link_joint" type="prismatic">
-      <limit lower="0.00000" upper="0.20000" effort="10.0" velocity="10.0"/>
+      <limit lower="-0.001" upper="0.20000" effort="100.0" velocity="1.0"/>
       <dynamics damping="10.0" friction="10.0"/>
       <origin rpy="3.14159 1.5708 -3.14159" xyz="-0.34568 0.00059 0.07033"/>

Commit message: lo arreglé mientras me comía una galleta y no he sentido tanta felicidad este mes

File: practica3/src/rover_kachau/urdf/arm/gripper.urdf.xacro (robot description, xacro)
@@ -1,89 +1,89 @@
 <?xml version="1.0"?>
 <robot xmlns:xacro="http://www.ros.org/wiki/xacro">
-  <xacro:macro name="gripper" params="prefix parent_link">
-    <joint name="${prefix}_pris_link4_link_joint" type="prismatic">
-      <limit lower="-0.130" upper="2" effort="10.0" velocity="10.0"/>
-      <dynamics damping="50.0" friction="10.0"/>
-      <origin rpy="3.14159 0 -1.5708" xyz="0 0 0"/>
-      <parent link="${parent_link}"/>
-      <child link="${prefix}_pris_link4_link"/>
-      <axis xyz="0 0 1"/>
-    </joint>
-    <joint name="${prefix}_pris_link4.001_link_joint" type="prismatic">
-      <limit lower="0.00000" upper="0.20000" effort="100.0" velocity="1.0"/>
-      <dynamics damping="10.0" friction="10.0"/>
-      <origin rpy="0 1.5708 3.14159" xyz="0.34568 0.00059 0.07033"/>
-      <parent link="${prefix}_pris_link4_link"/>
-      <child link="${prefix}_pris_link4.001_link"/>
-      <axis xyz="0 0 1"/>
-    </joint>
-    <joint name="${prefix}_pris_link4.002_link_joint" type="prismatic">
-      <limit lower="-0.001" upper="0.20000" effort="100.0" velocity="1.0"/>
-      <dynamics damping="10.0" friction="10.0"/>
-      <origin rpy="3.14159 1.5708 -3.14159" xyz="-0.34568 0.00059 0.07033"/>
-      <parent link="${prefix}_pris_link4_link"/>
-      <child link="${prefix}_pris_link4.002_link"/>
-      <axis xyz="0 0 1"/>
-    </joint>
-    <link name="${prefix}_pris_link4_link">
-      <collision name="pris_link4_collision">
-        <origin rpy="-3.14159 0 0" xyz="0 0 0"/>
-        <geometry>
-          <mesh filename="package://rover_kachau/meshes/dae/Cylinder.013.dae" scale="0.03922 0.03922 0.61477"/>
-        </geometry>
-      </collision>
-      <inertial>
-        <inertia ixx="0.00071" ixy="0.00000" ixz="-0.00000" iyy="0.00072" iyz="0.00000" izz="0.00001"/>
-        <origin rpy="0 0 0" xyz="0 0 0"/>
-        <mass value="0.00100"/>
-      </inertial>
-      <visual name="pris_link4">
-        <material name="Material.004"/>
-        <origin rpy="-3.14159 0 0" xyz="0 0 0"/>
-        <geometry>
-          <mesh filename="package://rover_kachau/meshes/dae/Cylinder.013.dae" scale="0.03922 0.03922 0.61477"/>
-        </geometry>
-      </visual>
-    </link>
-    <link name="${prefix}_pris_link4.001_link">
-      <collision name="pris_link4.001_collision">
-        <origin rpy="0 0 0" xyz="0 0 0"/>
-        <geometry>
-          <box size="0.02510 0.06000 0.09410"/>
-        </geometry>
-      </collision>
-      <inertial>
-        <inertia ixx="0.00052" ixy="0.00000" ixz="0.00000" iyy="0.00040" iyz="0.00000" izz="0.00018"/>
-        <origin rpy="0 0 0" xyz="0 0 0"/>
-        <mass value="0.50000"/>
-      </inertial>
-      <visual name="pris_link4.001">
-        <material name="Material.003"/>
-        <origin rpy="0 -1.5708 0" xyz="0 0 0"/>
-        <geometry>
-          <mesh filename="package://rover_kachau/meshes/dae/Cylinder.009.dae" scale="0.03922 0.03922 0.61477"/>
-        </geometry>
-      </visual>
-    </link>
-    <link name="${prefix}_pris_link4.002_link">
-      <collision name="pris_link4.002_collision">
-        <origin rpy="0 -1.5708 3.14159" xyz="0 0 0"/>
-        <geometry>
-          <box size="0.02510 0.06000 0.09410"/>
-        </geometry>
-      </collision>
-      <inertial>
-        <inertia ixx="0.00052" ixy="-0.00000" ixz="0.00000" iyy="0.00040" iyz="-0.00000" izz="0.00018"/>
-        <origin rpy="0 0 0" xyz="0 0 0"/>
-        <mass value="0.00100"/>
-      </inertial>
-      <visual name="pris_link4.002">
-        <material name="Material.004"/>
-        <origin rpy="0 -1.5708 3.14159" xyz="0 0 0"/>
-        <geometry>
-          <mesh filename="package://rover_kachau/meshes/dae/Cylinder.010.dae" scale="0.03922 0.03922 0.61477"/>
-        </geometry>
-      </visual>
-    </link>
-  </xacro:macro>
+<xacro:macro name="gripper" params="prefix parent_link">
+  <joint name="${prefix}_pris_link4_link_joint" type="prismatic">
+    <limit lower="-0.130" upper="2" effort="100.0" velocity="10.0"/>
+    <dynamics damping="5.0" friction="1.0"/>
+    <origin rpy="3.14159 0 -1.5708" xyz="0 0 0"/>
+    <parent link="${parent_link}"/>
+    <child link="${prefix}_pris_link4_link"/>
+    <axis xyz="0 0 1"/>
+  </joint>
+  <joint name="${prefix}_pris_link4.001_link_joint" type="prismatic">
+    <limit lower="0.00000" upper="0.20000" effort="100.0" velocity="1.0"/>
+    <dynamics damping="10.0" friction="10.0"/>
+    <origin rpy="0 1.5708 3.14159" xyz="0.34568 0.00059 0.07033"/>
+    <parent link="${prefix}_pris_link4_link"/>
+    <child link="${prefix}_pris_link4.001_link"/>
+    <axis xyz="0 0 1"/>
+  </joint>
+  <joint name="${prefix}_pris_link4.002_link_joint" type="prismatic">
+    <limit lower="-0.001" upper="0.20000" effort="100.0" velocity="1.0"/>
+    <dynamics damping="10.0" friction="10.0"/>
+    <origin rpy="3.14159 1.5708 -3.14159" xyz="-0.34568 0.00059 0.07033"/>
+    <parent link="${prefix}_pris_link4_link"/>
+    <child link="${prefix}_pris_link4.002_link"/>
+    <axis xyz="0 0 1"/>
+  </joint>
+  <link name="${prefix}_pris_link4_link">
+    <collision name="pris_link4_collision">
+      <origin rpy="-3.14159 0 0" xyz="0 0 0"/>
+      <geometry>
+        <mesh filename="package://rover_kachau/meshes/dae/Cylinder.013.dae" scale="0.03922 0.03922 0.61477"/>
+      </geometry>
+    </collision>
+    <inertial>
+      <inertia ixx="0.00071" ixy="0.00000" ixz="-0.00000" iyy="0.00072" iyz="0.00000" izz="0.00001"/>
+      <origin rpy="0 0 0" xyz="0 0 0"/>
+      <mass value="0.00100"/>
+    </inertial>
+    <visual name="pris_link4">
+      <material name="Material.004"/>
+      <origin rpy="-3.14159 0 0" xyz="0 0 0"/>
+      <geometry>
+        <mesh filename="package://rover_kachau/meshes/dae/Cylinder.013.dae" scale="0.03922 0.03922 0.61477"/>
+      </geometry>
+    </visual>
+  </link>
+  <link name="${prefix}_pris_link4.001_link">
+    <collision name="pris_link4.001_collision">
+      <origin rpy="0 -1.5708 0" xyz="0 0 0"/>  <!-- alineado con el visual -->
+      <geometry>
+        <box size="0.02510 0.06000 0.09410"/>  <!-- orden original, rotación corrige los ejes -->
+      </geometry>
+    </collision>
+    <inertial>
+      <inertia ixx="0.00052" ixy="0.00000" ixz="0.00000" iyy="0.00040" iyz="0.00000" izz="0.00018"/>
+      <origin rpy="0 0 0" xyz="0 0 0"/>
+      <mass value="0.50000"/>
+    </inertial>
+    <visual name="pris_link4.001">
+      <material name="Material.003"/>
+      <origin rpy="0 -1.5708 0" xyz="0 0 0"/>
+      <geometry>
+        <mesh filename="package://rover_kachau/meshes/dae/Cylinder.009.dae" scale="0.03922 0.03922 0.61477"/>
+      </geometry>
+    </visual>
+  </link>
+  <link name="${prefix}_pris_link4.002_link">
+    <collision name="pris_link4.002_collision">
+      <origin rpy="0 -1.5708 3.14159" xyz="0 0 0"/>
+      <geometry>
+        <box size="0.02510 0.06000 0.09410"/>
+      </geometry>
+    </collision>
+    <inertial>
+      <inertia ixx="0.00052" ixy="-0.00000" ixz="0.00000" iyy="0.00040" iyz="-0.00000" izz="0.00018"/>
+      <origin rpy="0 0 0" xyz="0 0 0"/>
+      <mass value="0.00100"/>
+    </inertial>
+    <visual name="pris_link4.002">
+      <material name="Material.004"/>
+      <origin rpy="0 -1.5708 3.14159" xyz="0 0 0"/>
+      <geometry>
+        <mesh filename="package://rover_kachau/meshes/dae/Cylinder.010.dae" scale="0.03922 0.03922 0.61477"/>
+      </geometry>
+    </visual>
+  </link>
+</xacro:macro>
 </robot>

File: practica3/src/rover_kachau/urdf/ros2_control.urdf.xacro (robot description, xacro)
@@ -10,4 +10,5 @@
     <hardware>
       <plugin>gz_ros2_control/GazeboSimSystem</plugin>
+      <param name="position_proportional_gain">5.0</param>
     </hardware>
     <joint name="wheels__frontL_link_joint">
